Commit message: it at least spawns in properly

File: install/reaper_description/share/reaper_description/urdf/URDFassy.urdf (robot description, URDF)
Before this commit: robot URDFassy, 3 links, 2 joints
Links:
- added link left_track, mass 5.0; collision box size=1.0 0.1 0.1; visual box size=1.0 0.1 0.1
- added link right_track, mass 5.0; collision box size=1.0 0.1 0.1; visual box size=1.0 0.1 0.1
Joints:
- added joint left_track_joint: type revolute, parent Chassis, child left_track, origin xyz=0 0.260 -0.15 rpy=0 0 0, axis 0 1 0, limit lower=-1000 upper=1000 effort=10 velocity=10
- added joint right_track_joint: type revolute, parent Chassis, child right_track, origin xyz=0 -0.260 -0.15 rpy=0 0 0, axis 0 1 0, limit lower=-1000 upper=1000 effort=10 velocity=10

File: src/reaper_description/urdf/URDFassy.urdf (robot description, URDF)
Before this commit: robot URDFassy, 3 links, 2 joints
Links:
- added link left_track, mass 5.0; collision box size=1.0 0.1 0.1; visual box size=1.0 0.1 0.1
- added link right_track, mass 5.0; collision box size=1.0 0.1 0.1; visual box size=1.0 0.1 0.1
Joints:
- added joint left_track_joint: type continuous, parent Chassis, child left_track, origin xyz=0 0.260 -0.15 rpy=0 0 0, axis 0 1 0
- added joint right_track_joint: type continuous, parent Chassis, child right_track, origin xyz=0 -0.260 -0.15 rpy=0 0 0, axis 0 1 0

Commit message: Just need to adjust the rollers

File: install/reaper_description/share/reaper_description/urdf/URDFassy.urdf (robot description, URDF)
Before this commit: robot URDFassy_tracked, 5 links, 4 joints
Links:
- removed link left_track
- removed link right_track
- added link left_roller_1, mass 0.8; collision cylinder length=0.10 radius=0.155; visual cylinder length=0.10 radius=0.155
- added link left_roller_2, mass 0.8; collision cylinder length=0.10 radius=0.155; visual cylinder length=0.10 radius=0.155
- added link right_roller_1, mass 0.8; collision cylinder length=0.10 radius=0.155; visual cylinder length=0.10 radius=0.155
- added link right_roller_2, mass 0.8; collision cylinder length=0.10 radius=0.155; visual cylinder length=0.10 radius=0.155
Joints:
- removed joint left_track_joint
- removed joint right_track_joint
- added joint left_roller_1_joint: type continuous, parent Chassis, child left_roller_1, origin xyz=0.4 0.25 0 rpy=0 0 0, axis 0 1 0
- added joint left_roller_2_joint: type continuous, parent Chassis, child left_roller_2, origin xyz=-0.1 0.25 0 rpy=0 0 0, axis 0 1 0
- added joint right_roller_1_joint: type continuous, parent Chassis, child right_roller_1, origin xyz=0.4 -0.25 0 rpy=0 0 0, axis 0 1 0
- added joint right_roller_2_joint: type continuous, parent Chassis, child right_roller_2, origin xyz=-0.1 -0.25 0 rpy=0 0 0, axis 0 1 0

File: src/reaper_description/urdf/URDFassy.urdf (robot description, URDF)
Before this commit: robot URDFassy_tracked, 5 links, 4 joints
Links:
- removed link left_track
- removed link right_track
- added link left_roller_1, mass 0.8; collision cylinder length=0.10 radius=0.155; visual cylinder length=0.10 radius=0.155
- added link left_roller_2, mass 0.8; collision cylinder length=0.10 radius=0.155; visual cylinder length=0.10 radius=0.155
- added link right_roller_1, mass 0.8; collision cylinder length=0.10 radius=0.155; visual cylinder length=0.10 radius=0.155
- added link right_roller_2, mass 0.8; collision cylinder length=0.10 radius=0.155; visual cylinder length=0.10 radius=0.155
Joints:
- removed joint left_track_joint
- removed joint right_track_joint
- added joint left_roller_1_joint: type continuous, parent Chassis, child left_roller_1, origin xyz=0.4 0.25 0 rpy=0 0 0, axis 0 1 0
- added joint left_roller_2_joint: type continuous, parent Chassis, child left_roller_2, origin xyz=-0.1 0.25 0 rpy=0 0 0, axis 0 1 0
- added joint right_roller_1_joint: type continuous, parent Chassis, child right_roller_1, origin xyz=0.4 -0.25 0 rpy=0 0 0, axis 0 1 0
- added joint right_roller_2_joint: type continuous, parent Chassis, child right_roller_2, origin xyz=-0.1 -0.25 0 rpy=0 0 0, axis 0 1 0
